File: board.brd (EAGLE design)
At the start: 127 x 85.7 mm, 195 parts, among them J1 XEM6310, U1 AD8022ARMZ, U2 AD5754BREZ, U3 ADR420ARZ, U4 LT1175CS8-5PBF, U5 LT1763CS8-5PBF, U6 AD5754BREZ, U7 ADR420ARZ, U8 AD8022ARMZ, U9 AD8022ARMZ, X1 LTI-SASF54GT, X10 LTI-SASF54GT, X11 LTI-SASF54GT, X12 LTI-SASF54GT, X13 LTI-SASF54GT, X14 LTI-SASF54GT, X2 LTI-SASF54GT, X3 LTI-SASF54GT, X4 LTI-SASF54GT, X5 LTI-SASF54GT, X6 LTI-SASF54GT, X7 LTI-SASF54GT, X8 LTI-SASF54GT, X9 LTI-SASF54GT

Commit message: added some helpful pdfs
Parts:
- C35, C36: value 100uF -> 47uF
Changed lines of the file:
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@@
 <attribute name="NAME" x="95.40875" y="42.06875" size="1.27" layer="21" rot="R180"/>
 </element>
-<element name="C35" library="rcl" package="UD-4X5,8_NICHICON" value="100uF" x="88.265" y="82.2325" smashed="yes" rot="R90">
+<element name="C35" library="rcl" package="UD-4X5,8_NICHICON" value="47uF" x="88.265" y="82.2325" smashed="yes" rot="R90">
 <attribute name="NAME" x="85.725" y="80.3275" size="1.016" layer="25" rot="R90"/>
 <attribute name="VALUE" x="91.44" y="80.3275" size="1.016" layer="27" rot="R90"/>
 </element>
-<element name="C36" library="rcl" package="UD-4X5,8_NICHICON" value="100uF" x="97.79" y="82.2325" smashed="yes" rot="R90">
+<element name="C36" library="rcl" package="UD-4X5,8_NICHICON" value="47uF" x="97.79" y="82.2325" smashed="yes" rot="R90">
 <attribute name="NAME" x="95.25" y="80.3275" size="1.016" layer="25" rot="R90"/>
 <attribute name="VALUE" x="100.965" y="80.3275" size="1.016" layer="27" rot="R90"/>
