File: board.sch (EAGLE design)
At the start: 77 parts, among them IC1 MC78M12BDTG, IC2 MC79M05CDTG, IC3 MC78M05CDTG, IC4 MC79M12BDTG, IC6 TPS77033, IC7 TPS77025, J1 XEM6310, U1 AD8022ARMZ, U2 AD5754BREZ, U3 ADR421ARMZ, X1 BU-SMA-V, X2 BU-SMA-V, X3 BU-SMA-V, X4 BU-SMA-V, X5 BU-SMA-V, X6 BU-SMA-V

Commit message: Layout changes
Parts:
- removed U$2: KK3V, molex-kk:KK3V
Connections:
- net +15V: no longer U$2.1
- net -15V: no longer U$2.3
- net 0V: no longer U$2.2
- net GND: now also ADC1.DGND
- net GNDI: no longer ADC1.DGND
Changed lines of the file:
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@@
 <part name="VDD1" library="supply1" deviceset="VDD" device="" value="+2.5V"/>
 <part name="+3V1" library="supply1" deviceset="+3V3" device=""/>
-<part name="GNDI1" library="supply1" deviceset="GNDI" device=""/>
 <part name="IC2" library="linear" deviceset="MC79M" device="" technology="05CDTG" value="MC79M05CDTG"/>
 <part name="IC3" library="linear" deviceset="MC78M" device="" technology="05CDTG"/>
@@
 <part name="SH2" library="shorts" deviceset="SHORT-H" device="B5"/>
 <part name="GNDI5" library="supply1" deviceset="GNDI" device=""/>
-<part name="GND5" library="supply1" deviceset="0V" device=""/>
-<part name="U$2" library="molex-kk" deviceset="KK3*" device="V"/>
 <part name="GND6" library="supply1" deviceset="0V" device=""/>
 <part name="SUPPLY30" library="supply2" deviceset="GND" device=""/>
@@
 <part name="P+12" library="supply1" deviceset="+5V" device=""/>
 <part name="P-11" library="supply1" deviceset="-5V" device=""/>
-<part name="P+6" library="supply1" deviceset="+15V" device=""/>
-<part name="P-10" library="supply1" deviceset="-15V" device=""/>
 <part name="SUPPLY16" library="supply2" deviceset="+12V" device=""/>
 <part name="SUPPLY32" library="supply2" deviceset="-12V" device=""/>
@@
 <instance part="SH2" gate="G$1" x="7.62" y="73.66" rot="R270"/>
 <instance part="GNDI5" gate="G$1" x="7.62" y="86.36" rot="R180"/>
-<instance part="GND5" gate="1" x="-5.08" y="81.28" rot="R90"/>
-<instance part="U$2" gate="G$1" x="-22.86" y="81.28"/>
 <instance part="GND6" gate="1" x="7.62" y="66.04"/>
 <instance part="SUPPLY30" gate="GND" x="12.7" y="38.1"/>
@@
 <instance part="P+12" gate="1" x="162.56" y="60.96"/>
 <instance part="P-11" gate="1" x="162.56" y="20.32"/>
-<instance part="P+6" gate="1" x="-12.7" y="83.82" rot="R270"/>
-<instance part="P-10" gate="1" x="-12.7" y="78.74" rot="R90"/>
 <instance part="GND2" gate="1" x="7.62" y="-10.16" rot="R270"/>
 <instance part="C58" gate="G$1" x="86.36" y="-53.34" rot="R180"/>
@@
 </segment>
 <segment>
-<pinref part="GND5" gate="1" pin="0V"/>
-<pinref part="U$2" gate="G$1" pin="2"/>
-<wire x1="-17.78" y1="81.28" x2="-7.62" y2="81.28" width="0.1524" layer="91"/>
-</segment>
-<segment>
 <pinref part="SH2" gate="G$1" pin="P$2"/>
 <pinref part="GND6" gate="1" pin="0V"/>
@@
 </segment>
 <segment>
-<pinref part="U$2" gate="G$1" pin="1"/>
-<wire x1="-17.78" y1="83.82" x2="-15.24" y2="83.82" width="0.1524" layer="91"/>
-<pinref part="P+6" gate="1" pin="+15V"/>
-</segment>
-<segment>
 <pinref part="P+7" gate="1" pin="+15V"/>
 <pinref part="C32" gate="G$1" pin="2"/>
@@
 <junction x="-25.4" y="22.86"/>
 <pinref part="P-4" gate="1" pin="-15V"/>
-</segment>
-<segment>
-<pinref part="U$2" gate="G$1" pin="3"/>
-<wire x1="-17.78" y1="78.74" x2="-15.24" y2="78.74" width="0.1524" layer="91"/>
-<pinref part="P-10" gate="1" pin="-15V"/>
 </segment>
 <segment>
@@
 <attribute name="VALUE" x="132.08" y="198.12" size="1.778" layer="96" rot="R270"/>
 </instance>
-<instance part="GNDI1" gate="G$1" x="139.7" y="142.24"/>
 </instances>
 <busses>
@@
 <wire x1="144.78" y1="162.56" x2="137.16" y2="162.56" width="0.1524" layer="91"/>
 <wire x1="137.16" y1="165.1" x2="137.16" y2="162.56" width="0.1524" layer="91"/>
-<wire x1="137.16" y1="162.56" x2="137.16" y2="157.48" width="0.1524" layer="91"/>
+<wire x1="137.16" y1="162.56" x2="137.16" y2="160.02" width="0.1524" layer="91"/>
 <junction x="137.16" y="165.1"/>
 <junction x="137.16" y="162.56"/>
+<pinref part="ADC1" gate="A" pin="DGND"/>
+<wire x1="137.16" y1="160.02" x2="137.16" y2="157.48" width="0.1524" layer="91"/>
+<wire x1="137.16" y1="160.02" x2="144.78" y2="160.02" width="0.1524" layer="91"/>
+<junction x="137.16" y="160.02"/>
 </segment>
 <segment>
@@
 </segment>
 </net>
-<net name="GNDI" class="0">
-<segment>
-<pinref part="ADC1" gate="A" pin="DGND"/>
-<wire x1="144.78" y1="160.02" x2="139.7" y2="160.02" width="0.1524" layer="91"/>
-<wire x1="139.7" y1="160.02" x2="139.7" y2="144.78" width="0.1524" layer="91"/>
-<pinref part="GNDI1" gate="G$1" pin="GNDI"/>
-</segment>
-</net>

Commit message: Back to latest revision
Parts:
- removed C63, C64: 4.7uF, rcl:C-USC0603
- removed IC1: MC78M12BDTG, linear:MC78M12BDTG
- removed IC2: MC79M05CDTG, linear:MC79M05CDTG
- removed IC3: MC78M05CDTG, linear:MC78M05CDTG
- removed IC4: MC79M12BDTG, linear:MC79M12BDTG
- removed IC6: TPS77033, texas:TPS77033
- removed IC7: TPS77025, texas:TPS77025
- added ADC2: AD7357BRUZ, Analog Devices_By_element14_Batch_1:AD7357BRUZ
- added ADCOP3, ADCOP4: AD8138ARMZ, Analog Devices_By_element14_Batch_1:AD8138ARMZ
- added C29, C37, C39, C42, C43, C46, C48, C50, C52, C54, C56: 10uF, rcl:C-USC0603
- added C30: 0.1uF Tant, rcl:C-USC0603
- added C31: 0.01uF, rcl:C-USC0603
- added C36: 39pF, rcl:C-USC0603
- added C40, C41, C44, C45, C47, C49, C51, C53, C55, C57: 0.1uF, rcl:C-USC0603
- added R17: 115k, resistor:R-US_R0603
- added R18: 51k, resistor:R-US_R0603
- added R19: 130k, resistor:R-US_R0603
- added R20: 66k, resistor:R-US_R0603
- added R21, R22, R27, R28: 33, resistor:R-US_R0603
- added R23, R24, R25, R26, R29, R30, R31, R32: 499, resistor:R-US_R0603
- added R33, R34, R35, R36: 10K, resistor:R-US_R0603
- added SH3: SHORT-HB5, shorts:SHORT-HB5
- added U$1, U$2: LTM8045, adc:LTM8045
- added U$3: ADP222ACPZ-3325-R7, ADI-Phase-2:ADP222ACPZ-3325-R7
- added U$4, U$5, U$6, U$7: NFM31P, adc:NFM31P
- added U4: LT1175CS8-5PBF, LTC_By_element14_Batch_1:LT1175CS8-5PBF
- added U5: LT1763CS8-5PBF, LTC_By_element14_Batch_1:LT1763CS8-5PBF
- added U6: AD8022ARMZ, Analog Devices_By_element14_Batch_1:AD8022ARMZ
- added X7, X8: SMA-142-0701-871/876, con-coax:SMA-142-0701-871/876
- C25: value 10uF -> 100uF; device rcl:C-USC0603 -> rcl:C-USC1210
- C26: value 0.1uF -> 4.7uF
- C27: value 0.1uF -> 100uF; device rcl:C-USC0603 -> rcl:C-USC1210
- C28: value 10uF -> 4.7uF
- C33, C34: value 10uF -> 39pF
- C35: value 0.1uF -> 39pF
- J1: device opalkelly:XEM6310 -> adc:XEM6310
- U3: value ADR421ARMZ -> ADR420ARZ; device ADI-Phase-2:ADR421ARMZ -> Analog Devices_By_element14_Batch_1:ADR420ARZ
- X1, X2, X3, X4, X5, X6: value BU-SMA-V -> SMA-142-0701-871/876; device con-coax:BU-SMA-V -> con-coax:SMA-142-0701-871/876
Connections:
- removed net +12V: C33.2, C58.2, C59.2, IC1.VO, U2.AVDD, U3.VIN
- removed net +15V: C26.2, C32.2, IC1.VI, IC3.VI
- removed net -12V: C34.2, C60.2, C61.2, IC4.VO, U2.AVSS
- removed net -15V: C27.2, C35.2, IC2.VI, IC4.VI
- new net ADC10: ADC2.~CS
- new net ADC11: ADC2.SDATAB
- new net ADC12: ADC2.SDATAA
- new net ADC13: ADC2.SCLK
- new net GNDINT: C29.1, C30.1, SH1.P$1, SH2.P$1, SH3.P$1, U$3.EP, U$3.GND, U$6.2@1, U$6.2@2, U$7.2@1, U$7.2@2, U4.GND, U5.GND, U5.GND_2, U5.GND_3
- new net N$23: ADCOP3.-OUT, C33.2, R22.1, R24.2
- new net N$26: ADCOP3.-IN, C34.1, R23.1, R25.2
- new net N$27: U$2.RUN
- new net N$28: ADCOP3.+IN, C33.1, R24.1, R26.2
- new net N$29: U$1.RUN
- new net N$30: R19.2, U$2.RT
- new net N$32: R17.2, U$1.RT
- new net N$33: U$2.SYNC
- new net N$34: R18.2, U$1.FB
- new net N$35: C25.2, R18.1, U$1.VOUT+, U$4.1
- new net N$36: ADC2.VINA+, R21.2
- new net N$37: C27.1, R20.2, U$2.VOUT-, U$5.1
- new net N$38: R20.1, U$2.FB
- new net N$39: ADC2.VINA-, R22.2
- new net N$40: ADCOP3.+OUT, C34.2, R21.1, R23.2
- new net N$41: ADCOP4.-OUT, C35.2, R28.1, R30.2
- new net N$42: ADCOP4.-IN, C36.1, R29.1, R31.2
- new net N$43: ADCOP4.+IN, C35.1, R30.1, R32.2
- new net N$44: ADCOP4.+OUT, C36.2, R27.1, R29.2
- new net N$45: ADC2.VINB+, R27.2
- new net N$46: ADC2.VINB-, R28.2
- new net N$47: R32.1, X4.1
- new net N$48: U$5.3, U4.ILIM2, U4.ILIM4, U4.VIN, U4.VIN_2
- new net N$49: C31.1, U5.BYP
- new net N$51: R26.1, X3.1
- new net N$52: R33.1, U6.-IN2, U6.OUT2
- new net N$54: R34.1, U6.-IN1, U6.OUT1
- new net N$57: ADCOP3.VOCM, C45.2, R34.2, R36.2
- new net N$59: ADCOP4.VOCM, C44.1, R33.2, R35.1
- new net N$65: U$4.3, U5.IN, U5.~SHDN
- new net N$66: C30.2, U$6.1, U4.OUTPUT, U4.SENSE
- new net N$67: C29.2, C31.2, U$7.1, U5.OUT, U5.SENSE
- new net V+: C26.1, C28.1, U$1.V_IN, U$2.V_IN
- new net VREF2A: ADC2.REFA, C42.1, U6.+IN1
- new net VREF2B: ADC2.REFB, C43.1, U6.+IN2
- net +3V3: now also ADC2.VDR, C39.1, C40.1, U$3.SENSE1, U$3.VOUT1; no longer IC6.OUT
- net +5V: now also ADCOP3.V+, ADCOP4.V+, C32.1, C46.2, C47.2, C50.2, C51.2, C54.2, C55.2, C58.2, C59.2, U$3.EN1, U$3.EN2, U$3.VIN, U$7.3, U2.AVDD, U3.VIN, U6.+VS; no longer C25.2, C63.2, C64.2, IC3.VO, IC6.IN, IC7.IN
- net -5V: now also ADCOP3.V-, ADCOP4.V-, C48.2, C49.2, C52.2, C53.2, C56.2, C57.2, C60.2, C61.2, U$6.3, U2.AVSS, U6.-VS; no longer C28.2, IC2.VO
- net 0V: now also C26.2, C27.2, C28.2, R17.1, R19.1, SH1.P$2, U$1.GND, U$1.SYNC, U$1.VOUT-, U$2.GND, U$2.VOUT+, U$4.2@1, U$4.2@2, U$5.2@1, U$5.2@2; no longer C26.1, C27.1, C28.1, C32.1, C33.1, C34.1, C35.1, C63.1, C64.1, IC1.GND, IC2.GND, IC3.GND, IC4.GND, IC6.!EN, IC6.GND, IC7.!EN, IC7.GND, SH2.P$2
- net ADC0: now also ADC1.~CS, J1.P$170; no longer ADC1.SCLK, J1.P$24
- net ADC1: now also ADC1.SDATAB, J1.P$168; no longer ADC1.~CS, J1.P$23
- net ADC2: now also J1.P$166; no longer J1.P$22
- net ADC3: now also ADC1.SCLK, J1.P$164; no longer ADC1.SDATAB, J1.P$21
- net ADC4: now also J1.P$172; no longer J1.P$25
- net ADC5: now also J1.P$174; no longer J1.P$26
- net ADC6: now also J1.P$176; no longer J1.P$27
- net DACD0: now also J1.P$24; no longer J1.P$15
- net DACD1: now also J1.P$22; no longer J1.P$16
- net DACD2: now also J1.P$18; no longer J1.P$17
- net DACD3: now also J1.P$20; no longer J1.P$18
- net DACD4: now also J1.P$16; no longer J1.P$19
- net GND: now also ADC2.AGND, ADC2.AGND_2, ADC2.DGND, ADC2.REFGND, C32.2, C37.2, C39.2, C40.2, C41.2, C42.2, C43.2, C44.2, C45.1, C46.1, C47.1, C48.1, C49.1, C50.1, C51.1, C52.1, C53.1, C54.1, C55.1, C56.1, C57.1, R25.1, R31.1, R35.2, R36.1, SH3.P$2, X1.2, X2.2, X3.2, X4.2, X5.2, X6.2, X7.2, X8.2; no longer SH1.P$2, SH2.P$1, X1G$1.GND, X2G$1.GND, X3G$1.GND, X4G$1.GND, X5G$1.GND, X6G$1.GND
- net GNDI: now also SH2.P$2; no longer SH1.P$1
- net N$18: now also X7.1; no longer X5G$1.1
- net N$19: now also X6.1; no longer X4G$1.1
- net N$21: now also X8.1; no longer X6G$1.1
- net N$24: now also X2.1; no longer X2G$1.1
- net N$25: now also X1.1; no longer X1G$1.1
- net N$5: now also X5.1; no longer X3G$1.1
- net VDD: now also ADC2.VDD, C37.1, C41.1, U$3.SENSE2, U$3.VOUT2; no longer IC7.OUT
