File: board.sch (EAGLE design)
At the start: 79 parts, among them J1 XEM6310, U1 AD8022ARMZ, U2 AD5754BREZ, U3 ADR420ARZ, U4 LT1175CS8-5PBF, U5 LT1763CS8-5PBF, X1 LTI-SASF54GT, X2 LTI-SASF54GT, X5 LTI-SASF54GT, X6 LTI-SASF54GT, X7 LTI-SASF54GT, X8 LTI-SASF54GT

Commit message: More changes
Parts:
- added C33: 10uF, rcl:CPOL-US
- added C34: 0.1uF, rcl:C-USC0603
- added L1, L2: MPZ1608S601A, rcl:L-US
- C12, C13, C15, C17, C19, C21, C23, C29, C58, C60, C7, C8, C9: device rcl:C-USC0603 -> rcl:CPOL-US
Connections:
- new net N$27: L1.2, U$4.1
- new net N$41: L2.2, U$5.1
- net +3V3: now also C33.+, C34.1, C9.+; no longer C9.1
- net +5V: now also C17.+, C21.+, C58.+, C7.+; no longer C17.2, C21.2, C58.2, C7.2
- net -5V: now also C15.-, C19.-, C23.-, C60.-; no longer C15.2, C19.2, C23.2, C60.2
- net GND: now also C12.-, C13.-, C15.+, C17.-, C19.+, C21.-, C23.+, C29.+, C33.-, C34.2, C58.-, C60.+, C7.-, C8.-, C9.-; no longer C12.2, C13.2, C15.1, C17.1, C19.1, C21.1, C23.1, C29.1, C58.1, C60.1, C7.1, C8.2, C9.2
- net N$35: now also L1.1; no longer U$4.1
- net N$37: now also L2.1; no longer U$5.1
- net N$67: now also C29.-; no longer C29.2
- net V+: now also J1.P$101, J1.P$103, J1.P$105
- net VDD: now also C8.+; no longer C8.1
- net VREF1A: now also C12.+; no longer C12.1
- net VREF1B: now also C13.+; no longer C13.1
Other:
- moved on the sheet: C25, C27, U$4, U$5
